File: 01-SICk-CANary/01-SICk-CANary.kicad_pcb (KiCad board)
At the start: 2 copper layers, 45 x 30 mm, 37 parts, among them J1 Conn_01x06, J2 Conn_01x03, J3 Conn_01x03, Q1 Q_NMOS_DGS, Q2 Q_NMOS_DGS, SW1 SW_DPDT_x2, U1 TPD4E05U06DQA, U2 TJA1462AT/0Z

Commit message: feat: finish PCB design
Parts:
- D3, D4, D5, D6: value LED -> RED
- Q1, Q2: value Q_NMOS_DGS -> AO3400
- moved TP7 0.68 mm to (194.6, 96.2)
- moved TP8 0.68 mm to (194.6, 98.2)
- moved TP1 0.60 mm to (177.5, 91.0)
- moved TP3 0.60 mm to (180.9, 91.0)
- moved R5 0.17 mm to (178.2, 106.4)
- moved R6 0.17 mm to (178.2, 104.8), turned to 180 degrees
- moved D8 0.11 mm to (197.5, 91.9)
- moved R7 0.11 mm to (178.2, 109.6)
- moved R8 0.11 mm to (178.2, 108.0)
- moved J2 0.10 mm to (204.3, 93.7)
- moved R9 0.09 mm to (187.4, 94.9)
- moved D5 0.08 mm to (180.8, 109.6)
- moved D6 0.08 mm to (180.8, 108.0)
- moved D7 0.06 mm to (197.5, 105.1)
- moved J3 0.06 mm to (204.3, 106.9)
Connections:
- D7 pad 1: /CAN_P -> /CAN_N
- D7 pad 2: /CAN_N -> /CAN_P
- D8 pad 1: /CAN_P -> /CAN_N
- D8 pad 2: /CAN_N -> /CAN_P
- J2 pad 1: /CAN_P -> /CAN_N
- J2 pad 2: /CAN_N -> /CAN_P
- J3 pad 1: /CAN_P -> /CAN_N
- J3 pad 2: /CAN_N -> /CAN_P
Routing:
- net /CAN_P: track 0.00 -> 73.8 mm
- net /CAN_N: track 0.00 -> 73.6 mm
- net +VCC_IO: track 0.00 -> 28.7 mm, vias 0 -> 6
- net /STB: track 0.00 -> 24.6 mm
- net /CAN_RX: track 0.00 -> 19.4 mm
- net /CAN_TX: track 9.55 -> 28.7 mm
- net GND: track 0.00 -> 13.5 mm, vias 0 -> 14
- net +5V: track 0.00 -> 11.3 mm, vias 0 -> 7
- net Net-(Q2-S): track 0.00 -> 9.28 mm
- net Net-(Q1-S): track 0.00 -> 5.64 mm
- net /STB_R: track 0.00 -> 3.28 mm
- net Net-(C3-Pad1): track 0.00 -> 3.03 mm
- net Net-(SW1A-C): track 0.00 -> 2.35 mm
- net Net-(SW1B-C): track 0.00 -> 2.34 mm
- net /CAN_RXR: track 0.00 -> 1.61 mm
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- added copper zone on In2.Cu, net +5V
- added copper zone on In2.Cu, net +VCC_IO
- added copper zone on B.Cu, net GND
- added copper zone on F.Cu, net GND
- added copper zone on In1.Cu, net GND
- added copper zone on In2.Cu, net GND
Other:
- copper layers 2 -> 4
- board text added: "SICk CANary v1"
