File: 01-SICk-CANary/01-SICk-CANary.kicad_sch (KiCad schematic)
At the start: 37 parts, among them J1 Conn_01x06, J2 Conn_01x03, J3 Conn_01x03, Q1 Q_NMOS_DGS, Q2 Q_NMOS_DGS, SW1 SW_DPDT_x2, U1 TPD4E05U06DQA, U2 TJA1462AT/0Z

Commit message: chore: update board files
Parts:
- C1, C2: LCSC C1525 -> (none); MPN CL05B104KO5NNNC -> (none)
- C3: LCSC C576733 -> (none); MPN CC0402KRX7R0BB472 -> (none)
- D1, D2: LCSC C20611048 -> (none); MPN TSD05CDYFR -> (none)
- D3, D4, D5, D6: value LED -> RED; LCSC C2286 -> (none); MPN KT-0603R -> (none)
- D7, D8: LCSC C39832198 -> (none); MPN PESD2CANFD24V-TR -> (none)
- J1: LCSC C51940119 -> (none); MPN XY-SM06B-GHS-TB -> (none)
- J2, J3: LCSC C480579 -> (none); MPN 1840379 -> (none)
- Q1, Q2: value Q_NMOS_DGS -> AO3400; LCSC C20917 -> (none); MPN AO3400A -> (none)
- R1, R2, R3: LCSC C25092 -> (none); MPN 0402WGF220JTCE -> (none)
- R10, R9: LCSC C2481607 -> (none); MPN RK73H2ATTD60R4F -> (none)
- R4: LCSC C25744 -> (none); MPN 0402WGF1002TCE -> (none)
- R5, R6, R7, R8: LCSC C11702 -> (none); MPN 0402WGF1001TCE -> (none)
- SW1: LCSC C3664537 -> (none); MPN CAS-220A1 -> (none)
- TP1, TP2, TP3, TP4, TP5, TP6, TP7, TP8: now fitted; now in the parts list
- U1: LCSC C138714 -> (none); MPN TPD4E05U06DQAR -> (none)
- U2: LCSC C3234095 -> (none); MPN TJA1462AT/0Z -> (none)

Commit message: feat: finish PCB design
Connections:
- net CAN_N: now also D7.1, D8.1, J2.1 (Pin_1), J3.1 (Pin_1); no longer D7.2, D8.2, J2.2 (Pin_2), J3.2 (Pin_2)
- net CAN_P: now also D7.2, D8.2, J2.2 (Pin_2), J3.2 (Pin_2); no longer D7.1, D8.1, J2.1 (Pin_1), J3.1 (Pin_1)
